File: DSP_board/DSP_board/DSP_board.kicad_sch (KiCad schematic)
At the start: 39 parts, among them J7 Conn_02x10_Odd_Even, J8 Conn_02x06_Odd_Even, J9 Conn_02x06_Odd_Even

Commit message: header design
Parts:
- removed IC_dclink_leakage1: LM324DR, lm324:SOIC127P600X175-14N, symbol quad_opamp:LM324DR
- removed J7: Conn_02x10_Odd_Even, Connector_PinSocket_2.54mm:PinSocket_2x10_P2.54mm_Vertical, symbol Connector_Generic:Conn_02x10_Odd_Even
- removed J8: Conn_02x06_Odd_Even, Connector_PinSocket_2.54mm:PinSocket_2x07_P2.54mm_Vertical, symbol Connector_Generic:Conn_02x06_Odd_Even
- removed J9: Conn_02x06_Odd_Even, Connector_PinSocket_2.54mm:PinSocket_2x06_P2.54mm_Vertical, symbol Connector_Generic:Conn_02x06_Odd_Even
- added C12, C13, C20, C21, C22, C23, C24, C25, C26, C27, C28, C29, C30, C5, C6, C8: CAP, Capacitor_SMD:C_1206_3216Metric_Pad1.33x1.80mm_HandSolder, symbol pspice:CAP
- added C31, C32, C33: CAP, Capacitor_SMD:C_0805_2012Metric_Pad1.18x1.45mm_HandSolder, symbol pspice:CAP
- added IC_batt_2, IC_dc_link_leakage1: LM324DR, lm324:SOIC127P600X175-14N, symbol quad_opamp:LM324DR
- added J10, J8: Conn_02x01, Connector_PinSocket_2.54mm:PinSocket_1x02_P2.54mm_Vertical, symbol Connector_Generic:Conn_02x01
- added J7: Conn_02x12_Odd_Even, Connector_PinHeader_2.54mm:PinHeader_2x12_P2.54mm_Vertical, symbol Connector_Generic:Conn_02x12_Odd_Even
- added J9: Conn_01x05, Connector_PinSocket_2.54mm:PinSocket_1x05_P2.54mm_Vertical, symbol Connector_Generic:Conn_01x05
- added LDO1: NCV8114ASN165T1G, ldo_ncv118:SOT95P275X110-5N, symbol NCV8114ASN165T1G:NCV8114ASN165T1G
- added R53, R54, R55, R56, R57, R58, R59, R60, R61, R62, R63, R64, R65, R66, R67, R68, R69, R70, R71, R72, R73, R74, R75, R76, R77, R78: R, Resistor_SMD:R_1206_3216Metric_Pad1.30x1.75mm_HandSolder, symbol Device:R
- renumbered IC_offset1 to IC_batt_1
Connections:
- net I_leackage: now also C22.1, IC_dc_link_leakage1.14 (4OUT), R63.2
- net Igrid1: now also R19.2, J7.10 (Pin_10); no longer R26.2
- net Igrid1_sense: now also C14.1, IC_dc_link_leakage1.1 (1OUT), R54.2
- net Igrid2: now also J7.8 (Pin_8)
- net Igrid2_sense: now also C21.1, R60.2; no longer IC_grid23.13 (4IN-)
- net Igrid3: now also J7.6 (Pin_6)
- net Igrid3_sense: now also R36.2, C12.1; no longer IC_grid23.2 (1IN-)
- net OCD_grd2: now also J7.11 (Pin_11)
- net OCD_grid1: now also J7.12 (Pin_12)
- net OCD_grid3: now also J7.14 (Pin_14)
- net SCL: now also J7.24 (Pin_24)
- net SDA: now also J7.23 (Pin_23)
- net VSI11: now also J7.21 (Pin_21)
- net VSI12: now also J7.22 (Pin_22)
- net VSI21: now also J7.19 (Pin_19)
- net VSI22: now also J7.20 (Pin_20)
- net VSI31: now also J7.17 (Pin_17)
- net VSI32: now also J7.18 (Pin_18)
- net V_dc_link: now also J8.1 (Pin_1), R66.1; no longer R33.1
- net Vdc_link: now also C20.2, IC_dc_link_leakage1.8 (3OUT), R61.2, R64.1
- net Vgrid1: now also R25.1, J7.9 (Pin_9); no longer R29.1
- net Vgrid1_sense: now also C13.1, IC_dc_link_leakage1.7 (2OUT), R55.2
- net Vgrid2: now also J7.7 (Pin_7)
- net Vgrid2_sense: now also C15.2, R59.2, R62.1; no longer IC_grid23.9 (3IN-)
- net Vgrid3: now also J7.5 (Pin_5)
- net Vgrid3_sense: now also C11.1, R53.2; no longer IC_grid23.6 (2IN-)
- net batt_V_sense: now also IC_batt_1.1 (1OUT), IC_batt_1.2 (1IN-); no longer IC_batt_1.8 (3OUT), IC_batt_1.9 (3IN-)
- net batt_curr_0: now also J10.2 (Pin_2)
- net batt_curr_sense: now also C28.1, R74.2; no longer IC_batt_1.6 (2IN-)
- net batt_v: now also J10.1 (Pin_1)
- net ctrl_-15: now also C31.2, C32.2, C33.2, IC_batt_2.11 (GND), IC_dc_link_leakage1.11 (GND)
- net ctrl_15: now also C31.1, C32.1, C33.1, IC_batt_2.4 (VCC), IC_dc_link_leakage1.4 (VCC); no longer R13.2
- net ctrl_3v3: now also C27.1, LDO1.1 (IN), LDO1.3 (EN)
- net ctrl_gnd: now also C10.2, R26.1, R28.1, R29.1, R33.1, R35.1, C23.2, C26.2, C27.2, C29.1, C30.2, C8.2, J7.13 (Pin_13), LDO1.2 (GND), R59.1, R61.1, R65.1, R67.1, R69.1, R73.1, R76.1, R78.2; no longer C14.2, R15.2
- net curr_leakeage_i: now also J8.2 (Pin_2), R71.2; no longer R35.2
- net offset_v: now also R13.1, R15.1, C24.2, C25.2, C29.2, C5.2, C6.2, LDO1.5 (OUT), R68.1, R70.1, R72.1; no longer C10.2, C11.2, C15.2, IC_batt_1.1 (1OUT), IC_batt_1.2 (1IN-), R19.1, R25.1, R28.1, R36.1
- net vsi_fault: now also J7.15 (Pin_15)
- net vsi_ready: now also J7.16 (Pin_16)
- net at IC_batt_1.12 (4IN+): now also C30.1, R76.2, R77.2
- net ADC2: now reaches IC_batt_1.13 (4IN-)
- net ADC2: now also IC_batt_1.14 (4OUT)
- net at C7.1, IC_grid23.10 (3IN+), R16.2: now also R68.2; no longer R19.2
- new net: C6.1, IC_dc_link_leakage1.3 (1IN+), R15.2, R19.1
- new net: C5.1, IC_dc_link_leakage1.5 (2IN+), R13.2, R25.2
- new net: C8.1, IC_batt_2.3 (1IN+), R32.2, R56.2
- new net: C28.2, IC_batt_1.6 (2IN-), R74.1, R78.1
- new net: C25.1, IC_dc_link_leakage1.12 (4IN+), R71.1, R72.2
- new net: C23.1, IC_batt_2.12 (4IN+), R58.2, R65.2
- new net: C12.2, IC_grid23.2 (1IN-), R26.2, R36.1
- new net: C26.1, IC_batt_1.3 (1IN+), R73.2, R75.2
- new net: C13.2, IC_dc_link_leakage1.6 (2IN-), R35.2, R55.1
- new net: C10.1, IC_batt_2.5 (2IN+), R33.2, R57.2
- new net: C22.2, IC_dc_link_leakage1.13 (4IN-), R63.1, R69.2
- new net: C24.1, IC_dc_link_leakage1.10 (3IN+), R66.2, R70.2
- new net: C21.2, IC_grid23.13 (4IN-), R60.1, R67.2
- new net: C11.2, IC_grid23.6 (2IN-), R29.2, R53.1
- new net: C20.1, IC_dc_link_leakage1.9 (3IN-), R64.2
- new net: C14.2, IC_dc_link_leakage1.2 (1IN-), R28.2, R54.1
- new net: C15.1, IC_grid23.9 (3IN-), R62.2
- new net ADC1: IC_batt_1.8 (3OUT), IC_batt_1.9 (3IN-)
- new net ADC3: IC_batt_2.1 (1OUT), IC_batt_2.2 (1IN-)
- new net ADC4: IC_batt_2.6 (2IN-), IC_batt_2.7 (2OUT)
- new net ADC5: IC_batt_2.13 (4IN-), IC_batt_2.14 (4OUT)
- new net Analog_in1: J9.1 (Pin_1), R75.1
- new net Analog_in2: J9.2 (Pin_2), R77.1
- new net Analog_in3: J9.3 (Pin_3), R56.1
- new net Analog_in4: J9.4 (Pin_4), R57.1
- new net Analog_in5: J9.5 (Pin_5), R58.1
- new net relay_1: J7.4 (Pin_4)
- new net relay_2: J7.3 (Pin_3)
- new net relay_3: J7.1 (Pin_1)
Other:
- moved on the sheet: C1, C2, C3, C7, C9, IC_grid23, J_power1, R1, R16, R21, R23, R3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

Commit message: review changes
Parts:
- removed J10, J8: Conn_02x01, Connector_PinSocket_2.54mm:PinSocket_1x02_P2.54mm_Vertical, symbol Connector_Generic:Conn_02x01
- removed J7: Conn_02x12_Odd_Even, Connector_PinHeader_2.54mm:PinHeader_2x12_P2.54mm_Vertical, symbol Connector_Generic:Conn_02x12_Odd_Even
- removed J_power1: Conn_02x03_Counter_Clockwise, Connector_PinHeader_2.54mm:PinHeader_2x03_P2.54mm_Vertical, symbol Connector_Generic:Conn_02x03_Counter_Clockwise
- added C34, C35, C36, C38, C39, C40, C41, C42, C43, C44, C48: CAP, Capacitor_SMD:C_0603_1608Metric_Pad1.08x0.95mm_HandSolder, symbol pspice:CAP
- added C37, C49, C50: ESK107M050AG3EA, electrolytic_cap:CAPPRD350W60D800H1250, symbol electrolytic_cap:ESK107M050AG3EA
- added C45, C46, C47, C54, C55: CAP, Capacitor_SMD:C_0805_2012Metric_Pad1.18x1.45mm_HandSolder, symbol pspice:CAP
- added C51, C52, C53: CAP, Capacitor_SMD:C_1206_3216Metric_Pad1.33x1.80mm_HandSolder, symbol pspice:CAP
- added J10, J8: Conn_02x06_Odd_Even, Connector_PinSocket_2.54mm:PinSocket_2x06_P2.54mm_Vertical, symbol Connector_Generic:Conn_02x06_Odd_Even
- added J11, J12: Conn_02x05_Odd_Even, Connector_PinSocket_2.54mm:PinSocket_2x05_P2.54mm_Vertical, symbol Connector_Generic:Conn_02x05_Odd_Even
- added J13, J14, J15, J16: Conn_01x01_Female, Connector_PinSocket_2.54mm:PinSocket_1x01_P2.54mm_Vertical, symbol Connector:Conn_01x01_Female
- added J7: Conn_01x06, Connector_PinSocket_2.54mm:PinSocket_1x06_P2.54mm_Vertical, symbol Connector_Generic:Conn_01x06
- added R100, R101, R85, R91, R92, R93, R95, R96, R97, R98, R99: R, Resistor_SMD:R_0603_1608Metric_Pad0.98x0.95mm_HandSolder, symbol Device:R
Connections:
- net 24_gnd: now also J7.6 (Pin_6)
- net ADC1: now also IC_batt_1.1 (1OUT), IC_batt_1.2 (1IN-); no longer IC_batt_1.8 (3OUT), IC_batt_1.9 (3IN-)
- net DAB1PWM11: now also J8.6 (Pin_6)
- net DAB1PWM12: now also J8.5 (Pin_5)
- net DAB1PWM21: now also J8.4 (Pin_4)
- net DAB1PWM22: now also J8.3 (Pin_3)
- net DAB2_PWM11: now also J10.12 (Pin_12)
- net DAB2_PWM12: now also J10.11 (Pin_11)
- net DAB2_PWM21: now also J10.10 (Pin_10)
- net DAB2_PWM22: now also J10.9 (Pin_9)
- net I_leackage: now also R97.2
- net Igrid1: now also J11.3 (Pin_3)
- net Igrid1_sense: now also R99.2
- net Igrid2: now also J11.5 (Pin_5)
- net Igrid2_sense: now also R91.2
- net Igrid3: now also J11.1 (Pin_1)
- net Igrid3_sense: now also R93.2
- net OCD_grid1: now also J11.10 (Pin_10)
- net OCD_leakage: now also J8.11 (Pin_11)
- net SCL: now also J10.5 (Pin_5), J12.9 (Pin_9), J8.9 (Pin_9)
- net SDA: now also J10.6 (Pin_6), J12.7 (Pin_7), J8.10 (Pin_10)
- net VSI11: now also J12.10 (Pin_10)
- net VSI12: now also J12.8 (Pin_8)
- net VSI21: now also J12.6 (Pin_6)
- net VSI22: now also J12.4 (Pin_4)
- net VSI31: now also J12.2 (Pin_2)
- net VSI32: now also J12.1 (Pin_1)
- net V_12: now also J7.5 (Pin_5)
- net V_dc_link: now also J8.2 (Pin_2)
- net Vdc_link: now also R98.2
- net Vgrid1: now also J11.4 (Pin_4)
- net Vgrid1_sense: now also R96.2
- net Vgrid2: now also J11.6 (Pin_6)
- net Vgrid2_sense: now also R95.2
- net Vgrid3: now also J11.2 (Pin_2)
- net Vgrid3_sense: now also R92.2
- net batt_V_sense: now also IC_batt_1.8 (3OUT), IC_batt_1.9 (3IN-), R100.2; no longer IC_batt_1.1 (1OUT), IC_batt_1.2 (1IN-)
- net batt_curr_0: now also J10.1 (Pin_1)
- net batt_curr_sense: now also R101.2
- net batt_fault: now also J10.3 (Pin_3)
- net batt_ready: now also J10.4 (Pin_4)
- net batt_v: now also J10.2 (Pin_2)
- net ctrl_-15: now also C45.1, C46.1, C47.1, C49.1, C52.1, C55.1, J7.2 (Pin_2); no longer C31.2, C32.2, C33.2
- net ctrl_15: now also C37.1, C51.1, C54.1, J7.1 (Pin_1)
- net ctrl_3v3: now also C50.1, C53.1, J7.3 (Pin_3)
- net ctrl_gnd: now also C31.2, C32.2, C33.2, C34.1, C35.1, C36.1, C37.2, C38.1, C39.1, C40.1, C41.1, C42.1, C43.1, C44.1, C45.2, C46.2, C47.2, C48.1, C49.2, C50.2, C51.2, C52.2, C53.2, C54.2, C55.2, J10.8 (Pin_8), J11.7 (Pin_7), J13.1 (Pin_1), J14.1 (Pin_1), J15.1 (Pin_1), J16.1 (Pin_1), J7.4 (Pin_4), J8.12 (Pin_12)
- net curr_leakeage_i: now also J8.1 (Pin_1)
- net dc_fault: now also J8.7 (Pin_7)
- net dc_ready: now also J8.8 (Pin_8)
- net offset_v: now also R85.2
- net relay_1: now also J11.8 (Pin_8)
- net vsi_fault: now also J12.5 (Pin_5)
- net vsi_ready: now also J12.3 (Pin_3)
- new net I_leackage_f: C40.2, R97.1
- new net Igrid1_sense_f: C42.2, R99.1
- new net Igrid2_sense_f: C34.2, R91.1
- new net Igrid3_sense_f: C36.2, R93.1
- new net Vdc_link_f: C41.2, R98.1
- new net Vgrid1_sense_f: C39.2, R96.1
- new net Vgrid2_sense_f: C38.2, R95.1
- new net Vgrid3_sense_f: C35.2, R92.1
- new net batt_V_sense_f: C43.2, R100.1
- new net batt_curr_sense_f: C44.2, R101.1
- new net offset_f: C48.2, R85.1
Other:
- moved on the sheet: C31
