File: DSP_board/DSP_board/controller_sheet.kicad_sch (KiCad schematic)
At the start: 55 parts, among them IC1 SN74S1053NSR, IC5 F280025CPNQR, J1 Conn_01x02, J2 Conn_01x02, J3 Conn_01x02, J4 Conn_01x02, J5 1-84981-0, J6 Conn_01x02

Commit message: header design
Parts:
- added R79, R80, R81, R82, R83, R84, R85, R86, R87, R88, R89, R90: R, Resistor_SMD:R_1206_3216Metric_Pad1.30x1.75mm_HandSolder, symbol Device:R
Connections:
- net DAB1PWM11: now also B1.35 (IO32); no longer B1.63 (JA4)
- net DAB1PWM12: now also B1.34 (IO33); no longer B1.62 (JA3)
- net DAB1PWM21: now also B1.33 (IO34); no longer B1.61 (JA2)
- net DAB1PWM22: now also B1.32 (IO35); no longer B1.60 (JA1)
- net DAB2_PWM11: now also B1.31 (IO36); no longer B1.69 (JA10)
- net DAB2_PWM12: now also B1.30 (IO37); no longer B1.68 (JA9)
- net DAB2_PWM21: now also B1.29 (IO38); no longer B1.67 (JA8)
- net DAB2_PWM22: now also B1.28 (IO39); no longer B1.66 (JA7)
- net FPGA_3v3: no longer R10.2, R9.2
- net I_leackage: now also IC1.18 (D15), IC5.16 (A11C0); no longer IC1.17 (D14), IC5.15 (A14C4)
- net Igrid3_sense: now also IC1.14 (D11), IC5.12 (A3C5); no longer IC1.13 (D10), IC5.11 (C6)
- net OCD_grd2: now also B1.15 (A1), IC5.37 (GPIO11), R85.1; no longer B1.90 (JC7), IC5.78 (GPIO15)
- net OCD_grid1: now also B1.14 (A0), IC5.35 (GPIO13), R86.1; no longer B1.84 (JC1), IC5.79 (GPIO14)
- net OCD_grid3: now also B1.16 (A2), IC5.38 (GPIO33), R87.1; no longer B1.91 (JC8), IC5.77 (GPIO34)
- net OCD_leakage: now also B1.48 (IO11), IC5.77 (GPIO34), R82.2; no longer IC5.38 (GPIO33)
- net TDO: now also J5.3; no longer J5.4
- net TMS: now also J5.4; no longer J5.3
- net VSI11: now also B1.41 (IO28), R30.1; no longer B1.102 (JD7), R44.1
- net VSI12: now also B1.40 (IO27), R31.1; no longer B1.96 (JD1), R34.1
- net VSI21: now also B1.39 (IO28), R34.1; no longer B1.103 (JD8), R43.1
- net VSI22: now also B1.38 (IO29), R42.1; no longer B1.97 (JD2), R31.1
- net VSI31: now also B1.37 (IO30), R43.1; no longer B1.104 (JD9), R42.1
- net VSI32: now also B1.36 (IO31), R44.1; no longer B1.98 (JD3), R30.1
- net Vgrid1_sense: now also IC1.17 (D14), IC5.15 (A14C4); no longer IC1.18 (D15), IC5.16 (A11C0)
- net Vgrid2_sense: now also IC1.13 (D10), IC5.11 (C6); no longer IC1.15 (D12), IC5.13 (A2C9)
- net Vgrid3_sense: now also IC1.15 (D12), IC5.13 (A2C9); no longer IC1.14 (D11), IC5.12 (A3C5)
- net batt_fault: now also B1.27 (IO40)
- net batt_ready: now also B1.26 (IO41)
- net ctrl_3v3: now also R10.2, R9.2, R79.2
- net ctrl_gnd: now also R27.1, R80.1, R81.1, R82.1, R83.1, R84.1, R85.2, R86.2, R87.2, R88.1, R89.1, R90.1; no longer R27.2
- net dc_fault: now also B1.49 (IO10), IC5.78 (GPIO15), R81.2; no longer IC5.37 (GPIO11)
- net dc_ready: now also B1.50 (IO9), IC5.79 (GPIO14), R80.2; no longer IC5.35 (GPIO13)
- net en_dab: now also IC5.57 (GPIO42), R27.2; no longer IC5.56 (GPIO39), R27.1
- net en_vsi: now also IC5.56 (GPIO39); no longer IC5.57 (GPIO42)
- net offset_v: now also IC1.19 (D16); no longer IC1.8 (D07)
- net vsi_fault: now also B1.47 (IO12), R83.2; no longer B1.92 (JC10)
- net vsi_ready: now also B1.46 (IO13), R84.2; no longer B1.93 (JC10)
- net ADC1: now reaches IC5.23 (A7C3)
- net ADC2: now reaches IC5.24 (A8C11)
- net ADC3: now reaches IC5.27 (A4C14)
- net ADC4: now reaches IC5.28 (A9C8)
- net ADC5: now reaches IC5.29 (A10C10)
- net at IC5.5 (XRSN): now also R79.1
- net relay_3: now reaches IC5.67 (GPIO22)
- net relay_3: now also B1.17 (A3), R90.2
- net relay_2: now reaches IC5.68 (GPIO7)
- net relay_2: now also B1.18 (A4), R89.2
- net relay_1: now reaches IC5.69 (GPIO44)
- net relay_1: now also B1.19 (A5), R88.2
Other:
- moved on the sheet: IC1, R11, R12, R14, R17, R18, R20, R22, R24, R27, R30, R31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

Commit message: review changes
Parts:
- removed R85, R87, R89, R90: R, Resistor_SMD:R_1206_3216Metric_Pad1.30x1.75mm_HandSolder, symbol Device:R
Connections:
- net I_leackage: no longer IC5.16 (A11C0)
- net Igrid1_sense: no longer IC5.14 (A15C7)
- net Igrid2_sense: no longer IC5.10 (A6)
- net Igrid3_sense: no longer IC5.12 (A3C5)
- net Vdc_link: no longer IC5.17 (A5C2)
- net Vgrid1_sense: no longer IC5.15 (A14C4)
- net Vgrid2_sense: no longer IC5.11 (C6)
- net Vgrid3_sense: no longer IC5.13 (A2C9)
- net batt_V_sense: no longer IC5.19 (A0C15)
- net batt_curr_sense: no longer IC5.18 (A1)
- net offset_v: no longer IC5.22 (A12C1)
- net gpio30: now reaches IC5.1 (GPIO30)
- net gpio31: now reaches IC5.2 (GPIO31)
- net gpio25': now reaches IC5.42 (GPIO25)
- net gpio46': now reaches IC5.6 (GPIO46)
- net gpio3: now reaches IC5.60 (GPIO3)
- net gpio1: now reaches IC5.62 (GPIO1)
- net gpio40: now reaches IC5.64 (GPIO40)
- net gpio23: now reaches IC5.65 (GPIO23)
- net gpio41: now reaches IC5.66 (GPIO41)
- net gpio45: now reaches IC5.73 (GPIO45)
- net OCD_grd2: no longer names the net of B1.15 (A1)
- net OCD_grd2: no longer IC5.37 (GPIO11)
- net OCD_grid3: no longer names the net of B1.16 (A2)
- net OCD_grid3: no longer IC5.38 (GPIO33)
- net relay_2: no longer names the net of B1.18 (A4)
- net relay_2: no longer IC5.68 (GPIO7)
- net relay_3: no longer names the net of B1.17 (A3)
- net relay_3: no longer IC5.67 (GPIO22)
- new net I_leackage_f: IC5.16 (A11C0)
- new net Igrid1_sense_f: IC5.14 (A15C7)
- new net Igrid2_sense_f: IC5.10 (A6)
- new net Igrid3_sense_f: IC5.12 (A3C5)
- new net Vdc_link_f: IC5.17 (A5C2)
- new net Vgrid1_sense_f: IC5.15 (A14C4)
- new net Vgrid2_sense_f: IC5.11 (C6)
- new net Vgrid3_sense_f: IC5.13 (A2C9)
- new net batt_V_sense_f: IC5.19 (A0C15)
- new net batt_curr_sense_f: IC5.18 (A1)
- new net gpio11: IC5.37 (GPIO11)
- new net gpio22: IC5.67 (GPIO22)
- new net gpio33: IC5.38 (GPIO33)
- new net gpio7: IC5.68 (GPIO7)
- new net offset_f: IC5.22 (A12C1)
