File: aux_PS/aux_PS.kicad_pcb (KiCad board)
At the start: 2 copper layers, 15 parts, among them J1 P78E03-1000, J2 Conn_02x03_Counter_Clockwise

Commit message: controller_final
Other:
- board outline added: 92.2 x 69 mm
Changed lines of the file:
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@@
     (pad "2" smd rect (at 2.15 0 180) (size 1.6 2.8) (layers "F.Cu" "F.Paste" "F.Mask")
       (net 8 "24_gnd") (pintype "passive"))
-    (model "EEH-ZA1H100R.stp"
+    (model "${PROJECT_PATHS}/EEH-ZA1H100R.stp"
       (offset (xyz 0 0 0))
       (scale (xyz 1 1 1))
@@
     (pad "2" smd rect (at 2.15 0 180) (size 1.6 2.8) (layers "F.Cu" "F.Paste" "F.Mask")
       (net 8 "24_gnd") (pintype "passive"))
-    (model "EEH-ZA1H100R.stp"
+    (model "${PROJECT_PATHS}/EEH-ZA1H100R.stp"
       (offset (xyz 0 0 0))
       (scale (xyz 1 1 1))
@@
     (pad "4" thru_hole circle (at 45.72 0) (size 1.524 1.524) (drill 0.762) (layers *.Cu *.Mask)
       (net 3 "Net-(AC_DC1-Pad4)") (pinfunction "+Vo") (pintype "output"))
+    (model "${PROJECT_PATHS}/PSK-S6C-24.stp"
+      (offset (xyz 0 0 0))
+      (scale (xyz 1 1 1))
+      (rotate (xyz 180 0 0))
+    )
   )
   (footprint "PXO:PXO7812500S" (layer "F.Cu")
@@
     (pad "3" thru_hole circle (at 5.08 0 90) (size 1.5 1.5) (drill 1) (layers *.Cu *.Mask)
       (net 9 "V12") (pinfunction "VOUT") (pintype "passive"))
-    (model "PXO7812-500-S.stp"
+    (model "${PROJECT_PATHS}/PXO7812-500-S.stp"
       (offset (xyz 0 0 0))
       (scale (xyz 1 1 1))
@@
     (pad "4" thru_hole circle (at 45.72 0) (size 1.524 1.524) (drill 0.762) (layers *.Cu *.Mask)
       (net 6 "Net-(AC_DC2-Pad4)") (pinfunction "+Vo") (pintype "output"))
+    (model "${PROJECT_PATHS}/PSK-S6C-24.stp"
+      (offset (xyz 0 0 0))
+      (scale (xyz 1 1 1))
+      (rotate (xyz 180 0 0))
+    )
   )
   (footprint "Resistor_SMD:R_1206_3216Metric_Pad1.30x1.75mm_HandSolder" (layer "F.Cu")
@@
     (pad "3" thru_hole circle (at 5.08 0 180) (size 1.65 1.65) (drill 1.1) (layers *.Cu *.Mask)
       (net 13 "ctrl_3v3") (pinfunction "+VOUT") (pintype "passive"))
-    (model "P78E03-1000.stp"
+    (model "${PROJECT_PATHS}/P78E03-1000.stp"
       (offset (xyz 0 0 0))
       (scale (xyz 1 1 1))
@@
     (pad "23" thru_hole circle (at 0 0) (size 1.524 1.524) (drill 0.762) (layers *.Cu *.Mask)
       (net 7 "/V_24") (pinfunction "Vin") (pintype "input"))
+    (model "${PROJECT_PATHS}/DCWN06B-15.stp"
+      (offset (xyz -7.5 -9 0))
+      (scale (xyz 1 1 1))
+      (rotate (xyz 0 0 0))
+    )
   )
   (footprint "Connector_PinSocket_2.54mm:PinSocket_2x03_P2.54mm_Vertical" (layer "F.Cu")
@@
     )
   )
-  (gr_rect (start 58.17 42.98) (end 168.89 112.34) (layer "F.Fab") (width 0.1) (fill none))
+  (gr_rect (start 66.99 43.56) (end 159.15 112.51) (layer "Edge.Cuts") (width 0.1) (fill none))
   (segment (start 116.80114 71.30114) (end 116.80114 65.75886) (width 0.25) (layer "F.Cu") (net 3))
   (segment (start 118.29 64.27) (end 118.34 64.27) (width 0.25) (layer "F.Cu") (net 3))

Commit message: header design
Parts:
- added C6: 1u_cer, Capacitor_SMD:C_1206_3216Metric_Pad1.33x1.80mm_HandSolder, B.Cu at (118.8, 94.0)
- added C7: 1u_cer, Capacitor_SMD:C_1206_3216Metric_Pad1.33x1.80mm_HandSolder, B.Cu at (129.7, 94.0)
- added C8: 1u_cer, Capacitor_SMD:C_1206_3216Metric_Pad1.33x1.80mm_HandSolder, F.Cu at (119.3, 55.7)
- added C9: 1u_cer, Capacitor_SMD:C_1206_3216Metric_Pad1.33x1.80mm_HandSolder, B.Cu at (129.3, 100.8)
- added J3: Conn_01x06, Connector_PinSocket_2.54mm:PinSocket_1x06_P2.54mm_Vertical, F.Cu at (89.9, 52.0)
- added J4: Conn_01x01_Female, Connector:Banana_Jack_1Pin, F.Cu at (52.5, 109.8)
- added J5: Conn_01x01_Female, Connector:Banana_Jack_1Pin, F.Cu at (52.3, 92.0)
- added J6: Conn_01x01_Female, Connector:Banana_Jack_1Pin, F.Cu at (52.3, 73.2)
- added J7: Conn_01x01_Female, Connector:Banana_Jack_1Pin, F.Cu at (51.8, 56.8)
- added J8: Conn_01x06, Connector_PinSocket_2.54mm:PinSocket_1x06_P2.54mm_Vertical, F.Cu at (95.0, 121.7)
- AC_DC1, AC_DC2: footprint PSK-S6C-24:PSK-S6C-24 -> PSK-S6C-24:PSKS6C24
- C1, C2, R1, R2: moved to B.Cu
- DC_DC1: footprint DCWN-06B:DCWN-06B -> DCWN-06B:DCWN06B15
- J2: value Conn_02x03_Counter_Clockwise -> Conn_01x06; footprint Connector_PinSocket_2.54mm:PinSocket_2x03_P2.54mm_Vertical -> Connector_PinSocket_2.54mm:PinSocket_1x06_P2.54mm_Vertical
- moved J2 68.2 mm to (94.8, 114.4), turned to 90 degrees
- moved C3 37.0 mm to (108.9, 63.9), turned to -90 degrees
- moved C4 31.2 mm to (108.6, 92.3), turned to -90 degrees
- moved DC_DC1 25.4 mm to (124.1, 82.3)
- moved R1 24.4 mm to (120.6, 62.8), turned to 0 degrees
- moved C1 21.7 mm to (103.9, 64.2), turned to -90 degrees
- moved C2 21.7 mm to (103.5, 92.9), turned to -90 degrees
- moved PS1 20.6 mm to (116.6, 60.1), turned to 0 degrees
- moved D1 20.3 mm to (113.4, 87.6)
- moved AC_DC1 20.2 mm to (63.3, 87.5)
- moved C5 15.0 mm to (120.6, 65.2), turned to 0 degrees
- moved J1 13.9 mm to (125.6, 106.4), turned to 0 degrees
- moved AC_DC2 13.1 mm to (63.3, 59.0)
- moved D2 11.2 mm to (113.2, 64.8)
- moved R2 10.3 mm to (129.3, 103.2), turned to 0 degrees
Connections:
- AC_DC1 pad 1: unconnected-(AC_DC1-Pad1) -> Net-(AC_DC1-Pad1)
- AC_DC1 pad 2: unconnected-(AC_DC1-Pad2) -> Net-(AC_DC1-Pad2)
- AC_DC2 pad 1: unconnected-(AC_DC2-Pad1) -> Net-(AC_DC2-Pad1)
- AC_DC2 pad 2: unconnected-(AC_DC2-Pad2) -> Net-(AC_DC2-Pad2)
- D2 pad 1: 24_gnd -> Net-(AC_DC2-Pad4)
- J2 pad 4: ctrl_gnd -> V12
- J2 pad 6: V12 -> ctrl_gnd
Routing:
- net ctrl_-15: track 32.9 -> 127.9 mm
- net ctrl_15: track 27.5 -> 117.3 mm
- net ctrl_gnd: track 53.9 -> 133.8 mm
- net ctrl_3v3: track 41.7 -> 120.8 mm, vias 1 -> 0
- net V12: track 38.9 -> 107.5 mm, vias 0 -> 1
- net Net-(AC_DC1-Pad4): track 54.3 -> 11.5 mm, vias 1 -> 0
- net /V_24: track 71.0 -> 34.5 mm
- net Net-(AC_DC2-Pad4): track 43.6 -> 12.4 mm, vias 2 -> 0
- net Net-(AC_DC2-Pad2): track 0.00 -> 13.5 mm
- net Net-(AC_DC1-Pad1): track 0.00 -> 12.8 mm
- net Net-(AC_DC2-Pad1): track 0.00 -> 12.4 mm
- net Net-(AC_DC1-Pad2): track 0.00 -> 11.7 mm
- net 24_gnd: track 134.6 -> 140.2 mm
Other:
- board size 92.2 x 69 mm -> 93.3 x 74.5 mm

Commit message: review changes
Parts:
- removed J4, J5, J6, J7: Conn_01x01_Female, Connector:Banana_Jack_1Pin
- added C10: EEH-ZA1H100R, electro_cap:EEHZA1H100R, F.Cu at (130.3, 114.7)
- added C_ldo_i1: C, Capacitor_SMD:C_1206_3216Metric_Pad1.33x1.80mm_HandSolder, F.Cu at (123.6, 112.9)
- added U1: 1800408, power_connector:1800408, F.Cu at (48.7, 66.4)
- added U2: 1800408, power_connector:1800408, F.Cu at (48.8, 95.7)
- added U3: BA033CC0FP-E2, 3v3_ldo:ROHM_TO-252-3, B.Cu at (128.0, 120.3)
- moved J3 71.2 mm to (74.1, 121.4)
Connections:
- J2 pad 4: V12 -> ctrl_gnd
- J2 pad 5: 24_gnd -> V12
- J2 pad 6: ctrl_gnd -> 24_gnd
- J3 pad 4: V12 -> ctrl_gnd
- J3 pad 5: 24_gnd -> V12
- J3 pad 6: ctrl_gnd -> 24_gnd
- J8 pad 4: V12 -> ctrl_gnd
- J8 pad 5: 24_gnd -> V12
- J8 pad 6: ctrl_gnd -> 24_gnd
Routing:
- net ctrl_gnd: track 133.8 -> 16.4 mm, vias 0 -> 2
- net ctrl_-15: track 127.9 -> 75.3 mm
- net ctrl_3v3: track 120.8 -> 77.1 mm, vias 0 -> 1
- net ctrl_15: track 117.3 -> 105.1 mm, vias 0 -> 1
- net Net-(AC_DC1-Pad2): track 11.7 -> 23.3 mm
- net Net-(AC_DC2-Pad1): track 12.4 -> 19.5 mm
- net Net-(AC_DC1-Pad1): track 12.8 -> 19.7 mm
- net Net-(AC_DC2-Pad2): track 13.5 -> 17.9 mm
- net 24_gnd: track 140.2 -> 143.1 mm
- net V12: track 107.5 -> 109.5 mm
- added copper zone on B.Cu, net ctrl_gnd
Other:
- board size 93.3 x 74.5 mm -> 98.4 x 75.4 mm

Commit message: revie of power board
Routing:
- net 24_gnd: track 143.1 -> 6.77 mm, vias 2 -> 6
- net ctrl_15: track 105.1 -> 85.5 mm
- net V12: track 109.5 -> 100.6 mm
- net ctrl_gnd: track 16.4 -> 8.73 mm
- added copper zone on F.Cu, net 24_gnd
